Commit message: Update robot setup

File: descriptions/simple_car.urdf (robot description, URDF)
Before this commit: robot simple_car, 7 links, 6 joints
Links:
- added link imu, mass 0.001; collision box size=0.01 0.01 0.01; visual box size=0.01 0.01 0.01
- link base_link: geometry collision box size=0.5 0.25 0.15; visual box size=0.5 0.25 0.15
- link camera: geometry collision box size=0.03 0.03 0.05; visual box size=0.03 0.03 0.07
- link caster: geometry collision sphere radius=0.1; visual sphere radius=0.1
- link left_wheel: geometry collision cylinder length=0.05 radius=0.1; visual cylinder length=0.05 radius=0.1
- link lidar: geometry collision cylinder length=0.05 radius=0.05; visual cylinder length=0.05 radius=0.05
- link right_wheel: geometry collision cylinder length=0.05 radius=0.1; visual cylinder length=0.05 radius=0.1
Joints:
- added joint imu_joint: type fixed, parent base_link, child imu, origin xyz=0 0 0.2 rpy=0 0 0
- joint camera_joint: origin xyz=0.5 0 0.3 rpy=0 0 0 -> xyz=0.25 0 0.225 rpy=0 0 0
- joint caster_joint: origin xyz=0.3 0 0.15 rpy=0 0 0 -> xyz=0.17 0 0.1 rpy=0 0 0
- joint left_wheel_joint: origin xyz=-0.3 0.3 0.15 rpy=0 0 0 -> xyz=-0.17 0.15 0.1 rpy=0 0 0
- joint lidar_joint: origin xyz=0 0 0.4 rpy=0 0 0 -> xyz=0 0 0.28 rpy=0 0 0
- joint right_wheel_joint: origin xyz=-0.3 -0.3 0.15 rpy=0 0 0 -> xyz=-0.17 -0.15 0.1 rpy=0 0 0

Commit message: Update configs that remove drift (esp turning)

File: descriptions/simple_car.urdf (robot description, URDF)
Before this commit: robot simple_car, 8 links, 7 joints
Links:
- link imu: mass 0.001 -> None; geometry 
Joints:
- joint imu_joint: origin xyz=0 0 0.2 rpy=0 0 0 -> xyz=0 0 0.01 rpy=0 0 0
- joint left_wheel_joint: limit effort=50000 velocity=10 -> effort=50000 velocity=5
- joint right_wheel_joint: limit effort=50000 velocity=10 -> effort=50000 velocity=5

Commit message: Update speed and camera

File: descriptions/simple_car.urdf (robot description, URDF)
Before this commit: robot simple_car, 8 links, 7 joints
Joints:
- joint left_wheel_joint: limit effort=50000 velocity=5 -> effort=50000 velocity=10
- joint right_wheel_joint: limit effort=50000 velocity=5 -> effort=50000 velocity=10
